Commit message: Fixed Gazebo setup

File: baxter/baxter_description/urdf/baxter.urdf (robot description, URDF)
Before this commit: robot dv, 50 links, 49 joints
Links:
- link head: geometry collision sphere radius=0.001; visual mesh filename=package://baxter_description/meshes/head/H0.DAE
- link left_lower_elbow: geometry collision sphere radius=0.12; visual mesh filename=package://baxter_description/meshes/lower_elbow/E1.DAE
- link left_lower_forearm: geometry collision cylinder length=0.01 radius=0.12; visual mesh filename=package://baxter_description/meshes/lower_forearm/W1.DAE
- link left_lower_shoulder: geometry visual mesh filename=package://baxter_description/meshes/lower_shoulder/S1.DAE
- link left_upper_elbow: geometry collision cylinder length=0.05 radius=0.14; visual mesh filename=package://baxter_description/meshes/upper_elbow/E0.DAE
- link left_upper_forearm: geometry visual mesh filename=package://baxter_description/meshes/upper_forearm/W0.DAE
- link left_upper_shoulder: geometry collision cylinder length=0.22 radius=0.15; visual mesh filename=package://baxter_description/meshes/upper_shoulder/S0.DAE
- link left_wrist: geometry collision cylinder length=0.04 radius=0.12; visual mesh filename=package://baxter_description/meshes/wrist/W2.DAE
- link pedestal: geometry collision cylinder length=0.7 radius=0.25; visual mesh filename=package://baxter_description/meshes/base/PEDESTAL.DAE
- link right_lower_elbow: geometry collision sphere radius=0.12; visual mesh filename=package://baxter_description/meshes/lower_elbow/E1.DAE
- link right_lower_forearm: geometry collision cylinder length=0.01 radius=0.12; visual mesh filename=package://baxter_description/meshes/lower_forearm/W1.DAE
- link right_lower_shoulder: geometry visual mesh filename=package://baxter_description/meshes/lower_shoulder/S1.DAE
- link right_upper_elbow: geometry collision cylinder length=0.05 radius=0.14; visual mesh filename=package://baxter_description/meshes/upper_elbow/E0.DAE
- link right_upper_forearm: geometry visual mesh filename=package://baxter_description/meshes/upper_forearm/W0.DAE
- link right_upper_shoulder: geometry collision cylinder length=0.22 radius=0.15; visual mesh filename=package://baxter_description/meshes/upper_shoulder/S0.DAE
- link right_wrist: geometry collision cylinder length=0.04 radius=0.12; visual mesh filename=package://baxter_description/meshes/wrist/W2.DAE
- link screen: geometry collision sphere radius=0.001; visual mesh filename=package://baxter_description/meshes/head/H1.DAE
- link torso: geometry collision cylinder length=0.7 radius=0.27; visual mesh filename=package://baxter_description/meshes/torso/base_link.DAE

Commit message: Baxter stands up with color in Gazebo

File: baxter/baxter_description/urdf/baxter.urdf (robot description, URDF)
Before this commit: robot dv, 50 links, 49 joints
Links:
- removed link left_lower_elbow_highspeed_collision
- removed link left_lower_forearm_highspeed_collision
- removed link left_wrist_highspeed_collision
- removed link right_lower_elbow_highspeed_collision
- removed link right_lower_forearm_highspeed_collision
- removed link right_wrist_highspeed_collision
- link base: mass 10 -> 0.1
- link collision_head_link_1: mass 1.0 -> 0.001
- link collision_head_link_2: mass 1.0 -> 0.001
- link dummyhead1: mass 1.0 -> 0.001
- link head: mass 1 -> 0.547767
- link head_camera: mass 1.0 -> 0.001
- link left_arm_mount: mass 0.1 -> 0.001
- link left_gripper: mass 1.0 -> 0.001
- link left_hand_camera: mass 1.0 -> 0.001
- link left_hand_camera_axis: mass 1.0 -> 0.001
- link left_hand_range: mass 1.0 -> 0.001
- link left_torso_itb: mass 0.1 -> 0.001
- link left_upper_elbow_visual: mass 0.1 -> 0.001
- link left_upper_forearm_visual: mass 0.1 -> 0.001
- link pedestal: mass 5 -> 60.86397744; geometry collision mesh filename=package://baxter_description/meshes/base/PEDESTAL.DAE; visual mesh filename=package://baxter_description/meshes/base/PEDESTAL.DAE
- link right_arm_itb: mass 0.1 -> 0.001
- link right_arm_mount: mass 0.1 -> 0.001
- link right_gripper: mass 1.0 -> 0.001
- link right_hand_camera: mass 1.0 -> 0.001
- link right_hand_camera_axis: mass 1.0 -> 0.001
- link right_hand_range: mass 1.0 -> 0.001
- link right_torso_itb: mass 0.1 -> 0.001
- link right_upper_elbow_visual: mass 0.1 -> 0.001
- link right_upper_forearm_visual: mass 0.1 -> 0.001
- link screen: mass 1 -> 0.440171
- link sonar_ring: mass 1 -> 0.001
- link torso: mass 5 -> 35.336455
Joints:
- removed joint left_e1_fixed
- removed joint left_w1_fixed
- removed joint left_w2_fixed
- removed joint right_e1_fixed
- removed joint right_w1_fixed
- removed joint right_w2_fixed

Commit message: updates to urdf

File: baxter/baxter_description/urdf/baxter.urdf (robot description, URDF)
Before this commit: robot dv, 44 links, 43 joints
Links:
- link base: mass 0.1 -> 0.00094542
- link collision_head_link_1: mass 0.001 -> 0.00094542
- link collision_head_link_2: mass 0.001 -> 0.00094542
- link dummyhead1: mass 0.001 -> 0.00094542
- link head_camera: mass 0.001 -> 0.00094542
- link left_arm_itb: mass 0.1 -> 0.00094542
- link left_arm_mount: mass 0.001 -> 0.00094542
- link left_gripper: mass 0.001 -> 0.1
- link left_hand: geometry collision cylinder length=0.0464 radius=0.04
- link left_lower_elbow: geometry collision cylinder length=0.10 radius=0.06; visual mesh filename=package://baxter_description/meshes/lower_elbow/E1.DAE
- link left_lower_forearm: geometry collision cylinder length=0.10 radius=0.06; visual mesh filename=package://baxter_description/meshes/lower_forearm/W1.DAE
- link left_lower_shoulder: geometry collision cylinder length=0.12 radius=0.06; visual mesh filename=package://baxter_description/meshes/lower_shoulder/S1.DAE
- link left_torso_itb: mass 0.001 -> 0.00094542
- link left_upper_elbow: geometry collision cylinder length=0.107 radius=0.06; visual mesh filename=package://baxter_description/meshes/upper_elbow/E0.DAE
- link left_upper_elbow_visual: geometry collision cylinder length=0.273 radius=0.06
- link left_upper_forearm: geometry collision cylinder length=0.088 radius=0.06; visual mesh filename=package://baxter_description/meshes/upper_forearm/W0.DAE
- link left_upper_forearm_visual: geometry collision cylinder length=0.272 radius=0.06
- link left_upper_shoulder: geometry collision cylinder length=0.2722 radius=0.06; visual mesh filename=package://baxter_description/meshes/upper_shoulder/S0.DAE
- link left_wrist: geometry collision cylinder length=0.165 radius=0.06; visual mesh filename=package://baxter_description/meshes/wrist/W2.DAE
- link pedestal: geometry collision box size=0.92 0.83 0.3; visual mesh filename=package://baxter_description/meshes/base/PEDESTAL.DAE
- link right_arm_itb: mass 0.001 -> 0.00094542
- link right_arm_mount: mass 0.001 -> 0.00094542
- link right_gripper: mass 0.001 -> 0.1
- link right_hand: geometry collision cylinder length=0.0464 radius=0.04
- link right_lower_elbow: geometry collision cylinder length=0.10 radius=0.06; visual mesh filename=package://baxter_description/meshes/lower_elbow/E1.DAE
- link right_lower_forearm: geometry collision cylinder length=0.10 radius=0.06; visual mesh filename=package://baxter_description/meshes/lower_forearm/W1.DAE
- link right_lower_shoulder: geometry collision cylinder length=0.12 radius=0.06; visual mesh filename=package://baxter_description/meshes/lower_shoulder/S1.DAE
- link right_torso_itb: mass 0.001 -> 0.00094542
- link right_upper_elbow: geometry collision cylinder length=0.107 radius=0.06; visual mesh filename=package://baxter_description/meshes/upper_elbow/E0.DAE
- link right_upper_elbow_visual: geometry collision cylinder length=0.273 radius=0.06
- link right_upper_forearm: geometry collision cylinder length=0.088 radius=0.06; visual mesh filename=package://baxter_description/meshes/upper_forearm/W0.DAE
- link right_upper_forearm_visual: geometry collision cylinder length=0.272 radius=0.06
- link right_upper_shoulder: geometry collision cylinder length=0.2722 radius=0.06; visual mesh filename=package://baxter_description/meshes/upper_shoulder/S0.DAE
- link right_wrist: geometry collision cylinder length=0.165 radius=0.06; visual mesh filename=package://baxter_description/meshes/wrist/W2.DAE
- link sonar_ring: mass 0.001 -> 0.00094542

Commit message: Adding latest urdf updates in support of MoveIt.

File: baxter/baxter_description/urdf/baxter.urdf (robot description, URDF)
Before this commit: robot baxter, 50 links, 49 joints
Links:
- removed link left_lower_elbow_highspeed_collision
- removed link left_lower_forearm_highspeed_collision
- removed link left_wrist_highspeed_collision
- removed link right_lower_elbow_highspeed_collision
- removed link right_lower_forearm_highspeed_collision
- removed link right_wrist_highspeed_collision
- link base: mass 0 -> 0.00094542
- link collision_head_link_1: mass 0 -> 0.00094542
- link collision_head_link_2: mass 0 -> 0.00094542
- link dummyhead1: mass 0 -> 0.00094542
- link head: mass 0 -> 0.547767
- link head_camera: mass 0 -> 0.00094542
- link left_arm_itb: mass None -> 0.00094542
- link left_arm_mount: mass None -> 0.00094542
- link left_gripper: mass 0.0 -> 0.00094542
- link left_hand: geometry collision cylinder length=0.0464 radius=0.04
- link left_hand_camera: mass 0 -> 0.00094542
- link left_hand_camera_axis: mass 0 -> 0.00094542
- link left_hand_range: mass 0 -> 0.00094542
- link left_lower_elbow: geometry collision cylinder length=0.10 radius=0.06; visual mesh filename=package://baxter_description/meshes/lower_elbow/E1.STL
- link left_lower_forearm: geometry collision cylinder length=0.10 radius=0.06; visual mesh filename=package://baxter_description/meshes/lower_forearm/W1.STL
- link left_lower_shoulder: geometry collision cylinder length=0.12 radius=0.06; visual mesh filename=package://baxter_description/meshes/lower_shoulder/S1.STL
- link left_torso_itb: mass None -> 0.00094542
- link left_upper_elbow: geometry collision cylinder length=0.107 radius=0.06; visual mesh filename=package://baxter_description/meshes/upper_elbow/E0.STL
- link left_upper_elbow_visual: mass None -> 0.00094542; geometry collision cylinder length=0.273 radius=0.06
- link left_upper_forearm: geometry collision cylinder length=0.088 radius=0.06; visual mesh filename=package://baxter_description/meshes/upper_forearm/W0.STL
- link left_upper_forearm_visual: mass None -> 0.00094542; geometry collision cylinder length=0.272 radius=0.06
- link left_upper_shoulder: geometry collision cylinder length=0.2722 radius=0.06; visual mesh filename=package://baxter_description/meshes/upper_shoulder/S0.STL
- link left_wrist: geometry collision cylinder length=0.165 radius=0.06; visual mesh filename=package://baxter_description/meshes/wrist/W2.STL
- link pedestal: mass 0 -> 60.86397744; geometry collision box size=0.92 0.83 0.3; visual mesh filename=package://baxter_description/meshes/base/PEDESTAL.STL
- link right_arm_itb: mass None -> 0.00094542
- link right_arm_mount: mass None -> 0.00094542
- link right_gripper: mass 0.0 -> 0.00094542
- link right_hand: geometry collision cylinder length=0.0464 radius=0.04
- link right_hand_camera: mass 0 -> 0.00094542
- link right_hand_camera_axis: mass 0 -> 0.00094542
- link right_hand_range: mass 0 -> 0.00094542
- link right_lower_elbow: geometry collision cylinder length=0.10 radius=0.06; visual mesh filename=package://baxter_description/meshes/lower_elbow/E1.STL
- link right_lower_forearm: geometry collision cylinder length=0.10 radius=0.06; visual mesh filename=package://baxter_description/meshes/lower_forearm/W1.STL
- link right_lower_shoulder: geometry collision cylinder length=0.12 radius=0.06; visual mesh filename=package://baxter_description/meshes/lower_shoulder/S1.STL
- link right_torso_itb: mass None -> 0.00094542
- link right_upper_elbow: geometry collision cylinder length=0.107 radius=0.06; visual mesh filename=package://baxter_description/meshes/upper_elbow/E0.STL
- link right_upper_elbow_visual: mass None -> 0.00094542; geometry collision cylinder length=0.273 radius=0.06
- link right_upper_forearm: geometry collision cylinder length=0.088 radius=0.06; visual mesh filename=package://baxter_description/meshes/upper_forearm/W0.STL
- link right_upper_forearm_visual: mass None -> 0.00094542; geometry collision cylinder length=0.272 radius=0.06
- link right_upper_shoulder: geometry collision cylinder length=0.2722 radius=0.06; visual mesh filename=package://baxter_description/meshes/upper_shoulder/S0.STL
- link right_wrist: geometry collision cylinder length=0.165 radius=0.06; visual mesh filename=package://baxter_description/meshes/wrist/W2.STL
- link screen: mass 0 -> 0.440171
- link sonar_ring: mass 0 -> 0.00094542
- link torso: mass 0.000000 -> 35.336455
Joints:
- removed joint left_e1_fixed
- removed joint left_w1_fixed
- removed joint left_w2_fixed
- removed joint right_e1_fixed
- removed joint right_w1_fixed
- removed joint right_w2_fixed
- joint head_camera: origin xyz=0.12839 0.0 0.06368 rpy=1.9198622 0.0 1.571 -> xyz=0.12839 0.0 0.06368 rpy=1.9198622 0.0 1.57079632679
- joint head_nod: origin xyz=.088 0.0 0.0 rpy=1.9198622 0.0 1.571 -> xyz=.088 0.0 0.0 rpy=1.9198622 0.0 1.57079632679
- joint head_pan: limit lower=-1.571 upper=1.571 effort=50000 velocity=10000 -> lower=-1.57079632679 upper=1.57079632679 effort=50000 velocity=10000
- joint left_e0: origin xyz=0.102 0 0 rpy=1.571 0 1.571 -> xyz=0.102 0 0 rpy=1.57079632679 0 1.57079632679
- joint left_e0_fixed: origin xyz=0.107 0 0 rpy=1.571 0 1.571 -> xyz=0.107 0 0 rpy=1.57079632679 0 1.57079632679
- joint left_e1: origin xyz=0.069 0 0.26242 rpy=-1.571 -1.571 0 -> xyz=0.069 0 0.26242 rpy=-1.57079632679 -1.57079632679 0
- joint left_hand_range: origin xyz=0.032 -0.020245 0.0288 rpy=0 -1.571 -1.571 -> xyz=0.032 -0.020245 0.0288 rpy=0 -1.57079632679 -1.57079632679
- joint left_s1: origin xyz=0.069 0 0.27035 rpy=-1.571 0 0 -> xyz=0.069 0 0.27035 rpy=-1.57079632679 0 0
- joint left_torso_itb_fixed: origin xyz=-0.08897 0.15593 0.389125 rpy=-1.571 3.1415 0 -> xyz=-0.08897 0.15593 0.389125 rpy=-1.57079632679 3.1415 0
- joint left_w0: origin xyz=0.10359 0 0 rpy=1.571 0 1.571 -> xyz=0.10359 0 0 rpy=1.57079632679 0 1.57079632679
- joint left_w0_fixed: origin xyz=0.088 0 0 rpy=1.571 0 1.571 -> xyz=0.088 0 0 rpy=1.57079632679 0 1.57079632679
- joint left_w0_to_itb_fixed: origin xyz=-0.0565 0 0.12 rpy=-1.571 0 1.571 -> xyz=-0.0565 0 0.12 rpy=-1.57079632679 0 1.57079632679
- joint left_w1: limit lower=-1.571 upper=2.094 effort=20.0 velocity=5.0 -> lower=-1.57079632679 upper=2.094 effort=20.0 velocity=5.0; origin xyz=0.01 0 0.2707 rpy=-1.571 -1.571 0 -> xyz=0.01 0 0.2707 rpy=-1.57079632679 -1.57079632679 0
- joint left_w2: origin xyz=0.115975 0 0 rpy=1.571 0 1.571 -> xyz=0.115975 0 0 rpy=1.57079632679 0 1.57079632679
- joint right_e0: origin xyz=0.102 0 0 rpy=1.571 0 1.571 -> xyz=0.102 0 0 rpy=1.57079632679 0 1.57079632679
- joint right_e0_fixed: origin xyz=0.107 0 0 rpy=1.571 0 1.571 -> xyz=0.107 0 0 rpy=1.57079632679 0 1.57079632679
- joint right_e1: origin xyz=0.069 0 0.26242 rpy=-1.571 -1.571 0 -> xyz=0.069 0 0.26242 rpy=-1.57079632679 -1.57079632679 0
- joint right_hand_range: origin xyz=0.032 -0.020245 0.0288 rpy=0 -1.571 -1.571 -> xyz=0.032 -0.020245 0.0288 rpy=0 -1.57079632679 -1.57079632679
- joint right_s1: origin xyz=0.069 0 0.27035 rpy=-1.571 0 0 -> xyz=0.069 0 0.27035 rpy=-1.57079632679 0 0
- joint right_torso_itb_fixed: origin xyz=-0.08897 -0.15593 0.389125 rpy=1.571 0 0 -> xyz=-0.08897 -0.15593 0.389125 rpy=1.57079632679 0 0
- joint right_w0: origin xyz=0.10359 0 0 rpy=1.571 0 1.571 -> xyz=0.10359 0 0 rpy=1.57079632679 0 1.57079632679
- joint right_w0_fixed: origin xyz=0.088 0 0 rpy=1.571 0 1.571 -> xyz=0.088 0 0 rpy=1.57079632679 0 1.57079632679
- joint right_w0_to_itb_fixed: origin xyz=-0.0565 0 0.12 rpy=-1.571 0 1.571 -> xyz=-0.0565 0 0.12 rpy=-1.57079632679 0 1.57079632679
- joint right_w1: limit lower=-1.571 upper=2.094 effort=20.0 velocity=5.0 -> lower=-1.57079632679 upper=2.094 effort=20.0 velocity=5.0; origin xyz=0.01 0 0.2707 rpy=-1.571 -1.571 0 -> xyz=0.01 0 0.2707 rpy=-1.57079632679 -1.57079632679 0
- joint right_w2: origin xyz=0.115975 0 0 rpy=1.571 0 1.571 -> xyz=0.115975 0 0 rpy=1.57079632679 0 1.57079632679
